File: TP3.kicad_pcb (KiCad board)
At the start: 2 copper layers, 48 parts

Commit message: Puse un pin doble para Chf
Parts:
- removed C_HF2: ~, Connector_PinSocket_1.27mm:PinSocket_1x01_P1.27mm_Vertical
- C_HF1: value ~ -> Conn_01x02; footprint Connector_PinSocket_1.27mm:PinSocket_1x01_P1.27mm_Vertical -> Connector_PinSocket_2.54mm:PinSocket_1x02_P2.54mm_Vertical
- moved Vcc_12V1 39.2 mm to (88.4, 32.1)
- moved C_HF1 4.45 mm to (77.9, 32.1)
- moved Osc1 0.65 mm to (64.5, 51.1)
Connections:
- C_HF1 pad 1: Net-(I_Rga1-A) -> Net-(C_HF1-Pin_1)
- C_o1 pad 1: Net-(M_2-D) -> Net-(C_HF1-Pin_1)
- I_Rga1 pad 1: Net-(I_Rga1-A) -> Net-(C_HF1-Pin_2)
- I_Rgb1 pad 1: Net-(I_Rga1-A) -> Net-(C_HF1-Pin_2)
- Id_M1 pad 1: Net-(I_Rga1-A) -> Net-(C_HF1-Pin_2)
- Id_M2 pad 1: Net-(I_Rga1-A) -> Net-(C_HF1-Pin_2)
- Id_Mref1 pad 1: Net-(I_Rga1-A) -> Net-(C_HF1-Pin_2)
- M_2 pad 3: Net-(M_2-D) -> Net-(C_HF1-Pin_1)
- R_D2 pad 2: Net-(M_2-D) -> Net-(C_HF1-Pin_1)
- Vcc_12V1 pad 2: Net-(I_Rga1-A) -> Net-(C_HF1-Pin_2)
- Vd_M2 pad 1: Net-(M_2-D) -> Net-(C_HF1-Pin_1)
Other:
- board outline added: 95 x 95 mm

Commit message: Placa hecha, se usó una huella para C_c1 con las patas más separadas para hacer pasar la pista de la referencia
Parts:
- added J_Vin1: Jumper_2_Bridged, Connector_PinHeader_2.54mm:PinHeader_1x02_P2.54mm_Vertical, F.Cu at (185.0, 130.0)
- C_c1: footprint Capacitor_THT:CP_Radial_D10.0mm_P3.80mm -> Capacitor_THT:CP_Radial_D10.0mm_P7.50mm
- moved GND3 242.5 mm to (265.7, 139.4)
- moved C_g1 240.2 mm to (257.1, 146.3), turned to -90 degrees
- moved R_L1 238.8 mm to (259.8, 122.3), turned to -90 degrees
- moved R_G2b1 231.4 mm to (247.5, 131.4), turned to -90 degrees
- moved GND2 226.4 mm to (265.7, 85.1)
- moved J_RL1 219.8 mm to (259.2, 92.9)
- moved R_G1b1 218.7 mm to (247.4, 73.4), turned to -90 degrees
- moved Vg_M2 211.3 mm to (247.9, 124.0)
- moved R_D2 208.4 mm to (235.5, 73.9), turned to -90 degrees
- moved M_O2 202.2 mm to (234.3, 138.2), turned to 90 degrees
- moved M_2 199.5 mm to (235.7, 113.7), turned to 90 degrees
- moved RS2 199.2 mm to (236.9, 147.6), turned to 180 degrees
- moved R_G1b2 195.9 mm to (247.5, 87.0), turned to -90 degrees
- moved Vs_M2/Vd_Mo1 195.5 mm to (234.7, 124.0)
- moved Vs_Mo2 195.1 mm to (225.6, 147.3)
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- renumbered C_G1 to C_g1, Carga1 to J_RL1
Connections:
- C_i1 pad 1: Net-(V_in1-Pin_2) -> Net-(J_Vin1-A)
- Osc1 pad 1: GND -> /V_out
- Osc1 pad 2: /V_out -> GND
- V_in1 pad 1: GND -> Net-(J_Vin1-B)
- V_in1 pad 2: Net-(V_in1-Pin_2) -> GND
Routing:
- net Net-(C_HF1-Pin_2): track 0.00 -> 88.2 mm
- net Net-(M_2-G): track 0.00 -> 63.3 mm
- net Net-(C_HF1-Pin_1): track 0.00 -> 61.8 mm
- net /Vp: track 0.00 -> 52.0 mm
- net Net-(Id_Mref1-B): track 0.00 -> 48.2 mm
- net Net-(M_1-G): track 0.00 -> 43.1 mm
- net Net-(D_Etapa2-B): track 0.00 -> 37.7 mm
- net /V_out: track 0.00 -> 36.2 mm
- net Net-(M_1-S): track 0.00 -> 31.9 mm
- net Net-(D_Etapa1-A): track 0.00 -> 29.7 mm
- net Net-(M_O2-S): track 0.00 -> 22.7 mm
- net Net-(M_O1-S): track 0.00 -> 22.5 mm
- net Net-(J_Vin1-B): track 0.00 -> 17.8 mm
- net Net-(J_Vin1-A): track 0.00 -> 15.4 mm
- net Net-(J_RL1-A): track 0.00 -> 14.3 mm
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- added copper zone on B.Cu, net GND
Other:
- board size 95 x 95 mm -> 97.5 x 97.5 mm

Commit message: Se hizo el pdf para imprimir
Parts:
- added C_HF1: Conn_01x02, Connector_PinSocket_2.54mm:PinSocket_1x02_P2.54mm_Vertical, F.Cu at (79.2, 76.9)
- added C_c1: 470u, Capacitor_THT:CP_Radial_D10.0mm_P7.50mm, F.Cu at (65.6, 90.0)
- added C_g1: 100u, Capacitor_THT:CP_Radial_D8.0mm_P3.50mm, F.Cu at (111.0, 146.3)
- added C_i1: 10u, Capacitor_THT:CP_Radial_D5.0mm_P2.00mm, F.Cu at (34.2, 116.4)
- added C_o1: 10u, Capacitor_THT:CP_Radial_D5.0mm_P2.00mm, F.Cu at (111.3, 78.9)
- added C_s1: 100u, Capacitor_THT:CP_Radial_D8.0mm_P3.50mm, F.Cu at (50.3, 132.5)
- added D_Etapa1: Jumper_2_Bridged, Connector_PinHeader_2.54mm:PinHeader_1x02_P2.54mm_Vertical, F.Cu at (57.1, 100.8)
- added D_Etapa2: Jumper_2_Bridged, Connector_PinHeader_2.54mm:PinHeader_1x02_P2.54mm_Vertical, F.Cu at (81.3, 98.3)
- added GND1: TestPoint, Connector_PinHeader_2.54mm:PinHeader_1x01_P2.54mm_Vertical, F.Cu at (29.4, 77.6)
- added GND2: TestPoint, Connector_PinHeader_2.54mm:PinHeader_1x01_P2.54mm_Vertical, F.Cu at (119.6, 85.2)
- added GND3: TestPoint, Connector_PinHeader_2.54mm:PinHeader_1x01_P2.54mm_Vertical, F.Cu at (119.6, 139.5)
- added GND4: TestPoint, Connector_PinHeader_2.54mm:PinHeader_1x01_P2.54mm_Vertical, F.Cu at (29.4, 123.9)
- added I_Rga1: Jumper_2_Bridged, Connector_PinHeader_2.54mm:PinHeader_1x02_P2.54mm_Vertical, F.Cu at (35.8, 62.3)
- added I_Rgb1: Jumper_2_Bridged, Connector_PinHeader_2.54mm:PinHeader_1x02_P2.54mm_Vertical, F.Cu at (101.7, 62.3)
- added Id_M1: Jumper_2_Bridged, Connector_PinHeader_2.54mm:PinHeader_1x02_P2.54mm_Vertical, F.Cu at (50.0, 62.3)
- added Id_M2: Jumper_2_Bridged, Connector_PinHeader_2.54mm:PinHeader_1x02_P2.54mm_Vertical, F.Cu at (89.5, 62.3)
- added Id_Mref1: Jumper_2_Bridged, Connector_PinHeader_2.54mm:PinHeader_1x02_P2.54mm_Vertical, F.Cu at (69.2, 62.3)
- added J_RL1: Jumper_2_Bridged, Connector_PinHeader_2.54mm:PinHeader_1x02_P2.54mm_Vertical, F.Cu at (113.1, 93.0)
- added J_Vin1: Jumper_2_Bridged, Connector_PinHeader_2.54mm:PinHeader_1x02_P2.54mm_Vertical, F.Cu at (38.9, 130.1)
- added M_1: 2N7000, Package_TO_SOT_THT:TO-92_Inline_Wide, F.Cu at (56.7, 113.8)
- added M_2: 2N7000, Package_TO_SOT_THT:TO-92_Inline_Wide, F.Cu at (89.6, 113.8)
- added M_O1: 2N7000, Package_TO_SOT_THT:TO-92_Inline_Wide, F.Cu at (61.7, 138.2)
- added M_O2: 2N7000, Package_TO_SOT_THT:TO-92_Inline_Wide, F.Cu at (88.2, 138.2)
- added M_REF1: 2N7000, Package_TO_SOT_THT:TO-92_Inline_Wide, F.Cu at (75.0, 138.2)
- added Osc1: Conn_01x02, Connector_PinHeader_2.54mm:PinHeader_1x02_P2.54mm_Horizontal, F.Cu at (104.8, 108.7)
- added RS1: R_Potentiometer_Trim_US, Potentiometer_THT:Potentiometer_Bourns_3296W_Vertical, F.Cu at (63.7, 147.9)
- added RS2: R_Potentiometer_Trim_US, Potentiometer_THT:Potentiometer_Bourns_3296W_Vertical, F.Cu at (90.8, 147.7)
- added R_D1: 2,2k, Resistor_THT:R_Axial_DIN0207_L6.3mm_D2.5mm_P10.16mm_Horizontal, F.Cu at (50.3, 73.3)
- added R_D2: 1,5k, Resistor_THT:R_Axial_DIN0207_L6.3mm_D2.5mm_P10.16mm_Horizontal, F.Cu at (89.4, 74.0)
- added R_G1a1: 1M, Resistor_THT:R_Axial_DIN0207_L6.3mm_D2.5mm_P10.16mm_Horizontal, F.Cu at (35.8, 83.5)
- added R_G1a2: 1M, Resistor_THT:R_Axial_DIN0207_L6.3mm_D2.5mm_P10.16mm_Horizontal, F.Cu at (35.8, 97.2)
- added R_G1b1: 1M, Resistor_THT:R_Axial_DIN0207_L6.3mm_D2.5mm_P10.16mm_Horizontal, F.Cu at (101.4, 73.4)
- added R_G1b2: 1M, Resistor_THT:R_Axial_DIN0207_L6.3mm_D2.5mm_P10.16mm_Horizontal, F.Cu at (101.4, 87.1)
- added R_G2a1: 1M, Resistor_THT:R_Axial_DIN0207_L6.3mm_D2.5mm_P10.16mm_Horizontal, F.Cu at (44.7, 111.4)
- added R_G2b1: 1M, Resistor_THT:R_Axial_DIN0207_L6.3mm_D2.5mm_P10.16mm_Horizontal, F.Cu at (101.5, 131.5)
- added R_L1: 1k, Resistor_THT:R_Axial_DIN0207_L6.3mm_D2.5mm_P10.16mm_Horizontal, F.Cu at (113.7, 122.4)
- added R_REF2: R_Potentiometer_Trim_US, Potentiometer_THT:Potentiometer_Bourns_3296W_Vertical, F.Cu at (69.2, 110.6)
- added V_in1: Conn_01x02, Connector_PinHeader_2.54mm:PinHeader_1x02_P2.54mm_Horizontal, F.Cu at (43.7, 147.0)
- added Vcc_12V1: Conn_01x02, TerminalBlock:TerminalBlock_MaiXu_MX126-5.0-02P_1x02_P5.00mm, F.Cu at (118.2, 62.1)
- added Vd_M1: TestPoint, Connector_PinHeader_2.54mm:PinHeader_1x01_P2.54mm_Vertical, F.Cu at (50.5, 91.3)
- added Vd_M2: TestPoint, Connector_PinHeader_2.54mm:PinHeader_1x01_P2.54mm_Vertical, F.Cu at (89.5, 91.8)
- added Vg_M1: TestPoint, Connector_PinHeader_2.54mm:PinHeader_1x01_P2.54mm_Vertical, F.Cu at (32.2, 105.2)
- added Vg_M2: TestPoint, Connector_PinHeader_2.54mm:PinHeader_1x01_P2.54mm_Vertical, F.Cu at (101.8, 124.0)
- added Vs/Vg_Mref1: TestPoint, Connector_PinHeader_2.54mm:PinHeader_1x01_P2.54mm_Vertical, F.Cu at (74.4, 124.0)
- added Vs_M1/Vd_Mo1: TestPoint, Connector_PinHeader_2.54mm:PinHeader_1x01_P2.54mm_Vertical, F.Cu at (60.7, 124.0)
- added Vs_M2/Vd_Mo1: TestPoint, Connector_PinHeader_2.54mm:PinHeader_1x01_P2.54mm_Vertical, F.Cu at (88.6, 124.0)
- added Vs_Mo1: TestPoint, Connector_PinHeader_2.54mm:PinHeader_1x01_P2.54mm_Vertical, F.Cu at (53.0, 147.9)
- added Vs_Mo2: TestPoint, Connector_PinHeader_2.54mm:PinHeader_1x01_P2.54mm_Vertical, F.Cu at (79.5, 147.4)
- moved C_HF1 2.47 mm to (227.8, 76.9)
- moved C_c1 2.47 mm to (214.2, 90.0)
- moved C_g1 2.47 mm to (259.6, 146.3)
- moved C_i1 2.47 mm to (182.8, 116.3)
- moved C_o1 2.47 mm to (259.9, 78.8)
- moved C_s1 2.47 mm to (198.9, 132.4)
- moved D_Etapa1 2.47 mm to (205.7, 100.7)
- moved D_Etapa2 2.47 mm to (229.9, 98.2)
- moved GND1 2.47 mm to (178.0, 77.5)
- moved GND2 2.47 mm to (268.2, 85.1)
- moved GND3 2.47 mm to (268.2, 139.4)
- moved GND4 2.47 mm to (178.0, 123.8)
- moved I_Rga1 2.47 mm to (184.4, 62.2)
- moved I_Rgb1 2.47 mm to (250.3, 62.3)
- moved Id_M1 2.47 mm to (198.6, 62.3)
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Routing:
- net Net-(C_HF1-Pin_2): track 88.2 -> 176.4 mm
- net Net-(M_2-G): track 63.3 -> 126.6 mm
- net Net-(C_HF1-Pin_1): track 61.8 -> 123.5 mm
- net /Vp: track 52.0 -> 103.9 mm
- net Net-(Id_Mref1-B): track 48.2 -> 96.5 mm
- net Net-(M_1-G): track 43.1 -> 86.1 mm
- net Net-(D_Etapa2-B): track 37.7 -> 75.4 mm
- net /V_out: track 36.2 -> 72.5 mm
- net Net-(M_1-S): track 31.9 -> 63.8 mm
- net Net-(D_Etapa1-A): track 29.7 -> 59.3 mm
- net Net-(M_O2-S): track 22.7 -> 45.4 mm
- net Net-(M_O1-S): track 22.5 -> 44.9 mm
- net Net-(J_Vin1-B): track 17.8 -> 35.6 mm
- net Net-(J_Vin1-A): track 15.4 -> 30.9 mm
- net Net-(J_RL1-A): track 14.3 -> 28.5 mm
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Other:
- board size 97.5 x 97.5 mm -> 246.1 x 97.6 mm
